File: hardware/node/node.kicad_pcb (KiCad board)
At the start: 4 copper layers, 48.5 x 50 mm, 72 parts, among them J1 BOOT0_Jumper, J2 FTDI, J3 SMA Female, J4 2 x AA, J5 SWD, Q1 Si2323DDS, SW1 TVCM04N016BB, U1 RFM69HW, U2 SHTC3, U3 AT25DF512C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

Commit message: Use only resistors to ground to config unit #
Parts:
- removed R10, R6, R7, R8, R9: 4k7, Resistor_SMD:R_0603_1608Metric_Pad1.05x0.95mm_HandSolder
- moved R5 6.93 mm to (71.5, 53.0)
- moved R4 5.30 mm to (74.0, 53.0)
- moved R3 5.20 mm to (76.5, 53.0)
- moved R1 3.75 mm to (81.5, 53.0)
- moved R2 3.34 mm to (79.0, 53.0)
- moved R13 0.62 mm to (66.8, 53.0)
Connections:
- R1 pad 2: VCC -> GND
- R2 pad 1: /CONF0 -> /CONF1
- R3 pad 1: /CONF1 -> /CONF2
- R3 pad 2: VCC -> GND
- R4 pad 1: /CONF1 -> /CONF3
- R5 pad 1: /CONF2 -> /CONF4
- R5 pad 2: VCC -> GND
Routing:
- net VCC: track 54.2 -> 44.9 mm, vias 20 -> 15
- net GND: track 70.1 -> 66.0 mm, vias 19 -> 20
- net /CONF4: track 17.3 -> 15.1 mm
- net /CONF3: track 15.5 -> 13.5 mm
- net /CONF1: track 12.2 -> 10.5 mm
- net /CONF0: track 11.5 -> 10.0 mm
- net /CONF2: track 13.6 -> 12.1 mm
- net /BOOT0: track 26.2 -> 26.9 mm
Other:
- board text added: "Unit #"

Commit message: Changed switch
Parts:
- removed the G*** at (68.0, 85.0)
- J2: footprint Connector_PinHeader_2.54mm:PinHeader_1x06_P2.54mm_Vertical -> Connector_PinHeader_2.54mm:PinHeader_1x06_P2.54mm_Horizontal
- R1, R2, R3, R4, R5: value 4k7 -> 0
- SW1: value TVCM04N016BB -> DTSM-65R-V-B; footprint humidity:SW_TVCM04-N -> humidity:SW_SPST_DTSM-6
- moved TP2 15.7 mm to (58.6, 64.2), turned to 90 degrees
- moved C14 13.8 mm to (68.9, 71.5)
- moved R33 11.6 mm to (64.6, 71.5), turned to 0 degrees
- moved TP4 11.5 mm to (58.6, 67.2), turned to 90 degrees
- moved J2 9.70 mm to (60.8, 87.4)
- moved J1 7.99 mm to (67.5, 56.0), turned to 180 degrees
- moved R11 7.57 mm to (65.2, 75.1)
- moved R12 7.57 mm to (65.2, 81.1)
- moved R14 7.57 mm to (65.2, 77.1)
- moved R16 7.57 mm to (65.2, 79.1)
- moved R13 4.48 mm to (64.5, 56.9), turned to 270 degrees
- moved SW1 1.98 mm to (64.4, 65.2), turned to 270 degrees
Connections:
- SW1 pad 1: /STM_RESET -> Net-(SW1-Pad1)
- SW1 pad 2: Net-(SW1-Pad2) -> /STM_RESET
Routing:
- net /STM_RESET: track 25.1 -> 16.4 mm
- net /BOOT0: track 26.9 -> 19.0 mm
- net GND: track 66.0 -> 71.2 mm, vias 20 -> 18
- net /FTDI_RX: track 13.8 -> 10.5 mm
- net /USART2_RX: track 16.1 -> 17.3 mm
Other:
- board text added: "OOS 2019-06-07"
- board text removed: "2019-06-03"
- board text removed: "Olof Ohlsson Sax 2019-06-03"

Commit message: Changed to 22u bul caps
Parts:
- C12, C13: value C -> 18p
- C14: value 10n -> 100n
- C15, C5: value 100u -> 22u; footprint Capacitor_SMD:CP_Elec_6.3x5.3 -> Capacitor_SMD:CP_Elec_5x5.3
- R32: value 22k -> 10k
- U4: value STM32L031K6Tx -> STM32L031K6T6
- moved C5 2.38 mm to (91.9, 74.0), turned to 270 degrees
- moved C15 0.60 mm to (87.6, 95.2)
Routing:
- net GND: track 71.2 -> 96.9 mm
- net /RFM69_INT: track 23.1 -> 22.3 mm
- net VCC: track 44.8 -> 44.3 mm
- net /LEDG: track 25.2 -> 25.8 mm
