File: hardware/node-batteries/node-batteries.sch (KiCad schematic (older format))
At the start: 9 parts, among them J1 Conn_01x03_Male

Commit message: Added part numbers to node-batteries
Parts:
- BT1: TME Link (none) -> https://www.tme.eu/se/en/details/bh-311-1p/batteries-holder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; TME Price (none) -> 2.56888
- J1: TME Link (none) -> https://www.tme.eu/se/en/details/zl201-03g/pin-headers/conn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; TME Price (none) -> 0.22041
Changed lines of the file:
@@
 F 2 "humidity:AA_Battery_Holder" V 2600 3210 50  0001 C CNN
 F 3 "https://www.tme.eu/se/en/details/bh-311-1p/batteries-holders/comf/" V 2600 3210 50  0001 C CNN
+F 4 "https://www.tme.eu/se/en/details/bh-311-1p/batteries-holders/comf/" H 2600 3150 50  0001 C CNN "TME Link"
+F 5 "2.56888" H 2600 3150 50  0001 C CNN "TME Price"
 	1    2600 3150
 	1    0    0    -1
@@
 F 2 "Connector_PinSocket_2.54mm:PinSocket_1x03_P2.54mm_Vertical" H 3950 3300 50  0001 C CNN
 F 3 "~" H 3950 3300 50  0001 C CNN
+F 4 "https://www.tme.eu/se/en/details/zl201-03g/pin-headers/connfly/ds1021-1-3sf1-1/" H 3950 3300 50  0001 C CNN "TME Link"
+F 5 "0.22041" H 3950 3300 50  0001 C CNN "TME Price"
 	1    3950 3300
 	-1   0    0    -1

Commit message: Improved mounting holes and planes
Parts:
- MH1, MH2, MH3, MH4, MH5, MH6: footprint MountingHole:MountingHole_3.2mm_M3 -> humidity:MountingHole_3.2mm_M3
Changed lines of the file:
@@
 F 0 "MH1" H 5750 3296 50  0000 L CNN
 F 1 "MountingHole M3" H 5750 3205 50  0000 L CNN
-F 2 "MountingHole:MountingHole_3.2mm_M3" H 5650 3250 50  0001 C CNN
+F 2 "humidity:MountingHole_3.2mm_M3" H 5650 3250 50  0001 C CNN
 F 3 "~" H 5650 3250 50  0001 C CNN
 	1    5650 3250
@@
 F 0 "MH2" H 5750 3496 50  0000 L CNN
 F 1 "MountingHole M3" H 5750 3405 50  0000 L CNN
-F 2 "MountingHole:MountingHole_3.2mm_M3" H 5650 3450 50  0001 C CNN
+F 2 "humidity:MountingHole_3.2mm_M3" H 5650 3450 50  0001 C CNN
 F 3 "~" H 5650 3450 50  0001 C CNN
 	1    5650 3450
@@
 F 0 "MH3" H 5750 3696 50  0000 L CNN
 F 1 "MountingHole M3" H 5750 3605 50  0000 L CNN
-F 2 "MountingHole:MountingHole_3.2mm_M3" H 5650 3650 50  0001 C CNN
+F 2 "humidity:MountingHole_3.2mm_M3" H 5650 3650 50  0001 C CNN
 F 3 "~" H 5650 3650 50  0001 C CNN
 	1    5650 3650
@@
 F 0 "MH4" H 5750 3896 50  0000 L CNN
 F 1 "MountingHole M3" H 5750 3805 50  0000 L CNN
-F 2 "MountingHole:MountingHole_3.2mm_M3" H 5650 3850 50  0001 C CNN
+F 2 "humidity:MountingHole_3.2mm_M3" H 5650 3850 50  0001 C CNN
 F 3 "~" H 5650 3850 50  0001 C CNN
 	1    5650 3850
@@
 F 0 "MH5" H 5750 4096 50  0000 L CNN
 F 1 "MountingHole M3" H 5750 4005 50  0000 L CNN
-F 2 "MountingHole:MountingHole_3.2mm_M3" H 5650 4050 50  0001 C CNN
+F 2 "humidity:MountingHole_3.2mm_M3" H 5650 4050 50  0001 C CNN
 F 3 "~" H 5650 4050 50  0001 C CNN
 	1    5650 4050
@@
 F 0 "MH6" H 5750 4296 50  0000 L CNN
 F 1 "MountingHole M3" H 5750 4205 50  0000 L CNN
-F 2 "MountingHole:MountingHole_3.2mm_M3" H 5650 4250 50  0001 C CNN
+F 2 "humidity:MountingHole_3.2mm_M3" H 5650 4250 50  0001 C CNN
 F 3 "~" H 5650 4250 50  0001 C CNN
 	1    5650 4250
