File: hardware/node-batteries/node-batteries.kicad_pcb (KiCad board)
At the start: 2 copper layers, 83 x 66 mm, 11 parts, among them J1 Conn_01x03_Male

Commit message: Add silkscreen for JLCPCB order number
Other:
- board text added: "JLCJLCJLCJLC"
Changed lines of the file:
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@@
   (general
     (thickness 1.6)
-    (drawings 84)
+    (drawings 85)
     (tracks 0)
     (zones 0)
@@
       (xy 0.0254 -0.041597)) (layer B.Cu) (width 0.01))
   )
+  (gr_text JLCJLCJLCJLC (at 90 91.75) (layer B.SilkS)
+    (effects (font (size 1 1) (thickness 0.2)) (justify mirror))
+  )
   (gr_line (start 41.5 100) (end 33.5 100) (layer Edge.Cuts) (width 0.15))
