File: hardware/gateway/gateway.sch (KiCad schematic (older format))
At the start: 36 parts, among them J1 FTDI, J2 Conn_Coaxial, J3 Raspberry_Pi_2_3, J4 TFT_Connector, SW1 Rotary_Encoder_Switch, U1 RFM69HW, U2 MCP7940N-xSN, Y1 32768 - 6pF

Commit message: Gateway schematic
Parts:
- removed D2: D_Schottky, symbol Device:D_Schottky
- added D3: BAT54.215, Package_TO_SOT_SMD:SOT-23, symbol humidity:D_Schottky_AncK
- BT1: value Battery_Cell -> KEYS3001; footprint (none) -> humidity:CR1216 Keystone 3001; TME Link (none) -> https://www.tme.eu/se/en/details/keys3001/batteries-holders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
- D1: renamed from D?; footprint (none) -> LED_SMD:LED_0805_2012Metric_Pad1.15x1.40mm_HandSolder
- D2: renamed from D1; footprint (none) -> LED_SMD:LED_0805_2012Metric_Pad1.15x1.40mm_HandSolder
- J1: footprint (none) -> Connector_PinHeader_2.54mm:PinHeader_1x06_P2.54mm_Vertical
- J2: footprint RF2-03E-T-00-50-G -> humidity:Adam_Tech_SMA_Female_RF2-19A
- J4: footprint (none) -> humidity:FPC Connector 22 pins XF2M22151AR100; TME Link (none) -> https://www.tme.eu/se/en/details/xf2m22151ar100/connectors-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
- Y1: footprint (none) -> humidity:Crystal LFXTAL016178; TME Link (none) -> https://www.tme.eu/se/en/details/32.768k-85smxr/smd-quartz-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
- gave numbers to parts that had none: 5
- renumbered R8 to R11, R9 to R14, R10 to R15
Other:
- moved on the sheet: BT1, R15

Commit message: Gateway PCB
Parts:
- removed J4: TFT_Connector, humidity:FPC Connector 22 pins XF2M22151AR100, symbol humidity:TFT_Connector
- removed R10: 0, Resistor_SMD:R_0805_2012Metric_Pad1.15x1.40mm_HandSolder, symbol Device:R
- removed R14: 91, Resistor_SMD:R_1206_3216Metric_Pad1.42x1.75mm_HandSolder, symbol Device:R
- removed R5, R6, R7: 10k, Resistor_SMD:R_0805_2012Metric_Pad1.15x1.40mm_HandSolder, symbol Device:R
- removed R9: DNP, Resistor_SMD:R_0805_2012Metric_Pad1.15x1.40mm_HandSolder, symbol Device:R
- removed SW1: Rotary_Encoder_Switch, symbol Device:Rotary_Encoder_Switch
- BT1: value KEYS3001 -> KEYS3000; footprint humidity:CR1216 Keystone 3001 -> humidity:CR1216_Keystone_3000; TME Link https://www.tme.eu/se/en/details/keys3001/batteries-holders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 -> https://www.tme.eu/se/en/details/keys3000/batteries-holders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
- J1: footprint Connector_PinHeader_2.54mm:PinHeader_1x06_P2.54mm_Vertical -> Connector_PinHeader_2.54mm:PinHeader_1x06_P2.54mm_Horizontal
- J3: footprint Connector_PinSocket_2.54mm:PinSocket_2x20_P2.54mm_Vertical -> Connector_PinSocket_2.54mm:PinSocket_2x20_P2.54mm_Vertical_SMD
Connections:
- net labels added: ANT, VBAT, VBAT_D, VBAT_IN, X1, X2
- net labels removed: +5V, ENC_A, ENC_B, ENC_SW, RFM_CS, RFM_MISO, RFM_MOSI, RFM_SCK, TFT_CE, TFT_MOMI, TFT_RESET, TFT_SCK
- wire segments 215 -> 129
- no-connect marks 17 -> 27
Other:
- note added: "CS"
- note added: "MISO"
- note added: "MOSI"
- note added: "SCK"
- note removed: "PI SPI1: CS2"
- note removed: "TFT: DEM 128128A TMH-PW-N"
- note removed: "Use SPI0 in LoSSI mode"
- moved on the sheet: BT1, C1, C2, C3, C4, C5, D1, D2, J2, J3, R11, R12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

Commit message: Added local 3V3 regulator
Parts:
- added C6: 1u, Capacitor_SMD:C_0805_2012Metric_Pad1.15x1.40mm_HandSolder, symbol Device:C
- added U3: AP130-xxY, Package_TO_SOT_SMD:SOT-89-3_Handsoldering, symbol humidity:AP130-xxY
- BT1: TME Price (none) -> 4.2504
- C1: value 100u -> 22u; footprint Capacitor_SMD:CP_Elec_6.3x5.7 -> Capacitor_SMD:CP_Elec_5x5.3; TME Link (none) -> https://www.tme.eu/se/en/details/sc1e226m05005vr/85degc-smd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; TME Price (none) -> 0.36794
- C2, C3, C4, C5: footprint Capacitor_SMD:C_0805_2012Metric_Pad1.15x1.40mm_HandSolder -> Capacitor_SMD:C_0603_1608Metric_Pad1.05x0.95mm_HandSolder
- D3: TME Price (none) -> 0.22899
- J2: TME Link (none) -> https://www.tme.eu/se/en/details/rf2-19a-t-00-50-g/sma-smb-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; TME Price (none) -> 10.86
- J3: TME Link (none) -> https://www.tme.eu/se/en/details/zl264-40dg/pin-headers/nin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; TME Price (none) -> 24.27
- R1, R11, R12, R13, R15, R2, R3, R4, R8: footprint Resistor_SMD:R_0805_2012Metric_Pad1.15x1.40mm_HandSolder -> Resistor_SMD:R_0603_1608Metric_Pad1.05x0.95mm_HandSolder
- U1: TME Link (none) -> https://www.tme.eu/se/en/details/rfm69hw-433s2/rf-modules/h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; TME Price (none) -> 29.94
- U2: TME Link (none) -> https://www.tme.eu/se/en/details/mcp7940n-i_sn/rtc-circuits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; TME Price (none) -> 7.56
- Y1: TME Price (none) -> 6.09368
Connections:
- net labels added: +3V3_PI, +3V3_REG, +5V_PI
- net labels removed: +3.3V
- wire segments 129 -> 134
- no-connect marks 27 -> 26
Other:
- moved on the sheet: C1

Commit message: Layout improvemnets
Parts:
- added C7: 100n, Capacitor_SMD:C_0603_1608Metric_Pad1.05x0.95mm_HandSolder, symbol Device:C
- added R5: 10k, Resistor_SMD:R_0603_1608Metric_Pad1.05x0.95mm_HandSolder, symbol Device:R
- D3: value BAT54.215 -> B0520LW-7-F; footprint Package_TO_SOT_SMD:SOT-23 -> Diode_SMD:D_SOD-123; symbol humidity:D_Schottky_AncK -> Device:D_Schottky; TME Link https://www.tme.eu/se/en/details/bat54.215/smd-schottky-dio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 -> https://www.tme.eu/se/en/details/b0520lw-7-f/smd-schottky-d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; TME Price 0.22899 -> 0.50890
- R1, R12, R13, R4: footprint Resistor_SMD:R_0603_1608Metric_Pad1.05x0.95mm_HandSolder -> humidity:R_0603_1608Metric_Pad1.05x0.95mm_HandSolder-DNP
Connections:
- net labels added: CS, MFP, MISO, MOSI, SCK
- wire segments 134 -> 139
- no-connect marks 26 -> 24
Other:
- note removed: "CS"
- note removed: "MISO"
- note removed: "MOSI"
- note removed: "SCK"
- moved on the sheet: BT1, R15
Changed lines of the file:
@@
 L Device:Battery_Cell BT1
 U 1 1 5CF7BB91
-P 8600 1300
-F 0 "BT1" V 8450 1300 50  0000 L CNN
-F 1 "KEYS3000" V 8800 1300 50  0000 C CNN
-F 2 "humidity:CR1216_Keystone_3000" V 8600 1360 50  0001 C CNN
-F 3 "~" V 8600 1360 50  0001 C CNN
-F 4 "https://www.tme.eu/se/en/details/keys3000/batteries-holders/keystone/3000/" V 8600 1300 50  0001 C CNN "TME Link"
-F 5 "4.2504" H 0   0   50  0001 C CNN "TME Price"
-	1    8600 1300
+P 9450 1300
+F 0 "BT1" V 9300 1300 50  0000 L CNN
+F 1 "KEYS3000" V 9650 1300 50  0000 C CNN
+F 2 "humidity:CR1216_Keystone_3000" V 9450 1360 50  0001 C CNN
+F 3 "~" V 9450 1360 50  0001 C CNN
+F 4 "https://www.tme.eu/se/en/details/keys3000/batteries-holders/keystone/3000/" V 9450 1300 50  0001 C CNN "TME Link"
+F 5 "4.2504" H 850 0   50  0001 C CNN "TME Price"
+	1    9450 1300
 	1    0    0    -1
 $EndComp
@@
 L Device:R R15
 U 1 1 5CF7BDA8
-P 7850 1400
-F 0 "R15" V 7950 1400 50  0000 C CNN
-F 1 "1k" V 7850 1400 50  0000 C CNN
-F 2 "Resistor_SMD:R_0603_1608Metric_Pad1.05x0.95mm_HandSolder" V 7780 1400 50  0001 C CNN
-F 3 "~" H 7850 1400 50  0001 C CNN
-	1    7850 1400
-	1    0    0    -1
-$EndComp
-Wire Wire Line
-	7850 1550 7850 1800
-Wire Wire Line
-	8600 1100 8600 900
+P 8450 900
+F 0 "R15" V 8550 900 50  0000 C CNN
+F 1 "1k" V 8450 900 50  0000 C CNN
+F 2 "Resistor_SMD:R_0603_1608Metric_Pad1.05x0.95mm_HandSolder" V 8380 900 50  0001 C CNN
+F 3 "~" H 8450 900 50  0001 C CNN
+	1    8450 900
+	0    1    1    0
+$EndComp
+Wire Wire Line
+	9450 1100 9450 900
 $Comp
 L power:GND #PWR025
 U 1 1 5CF7C329
-P 8600 1450
-F 0 "#PWR025" H 8600 1200 50  0001 C CNN
-F 1 "GND" H 8605 1277 50  0000 C CNN
-F 2 "" H 8600 1450 50  0001 C CNN
-F 3 "" H 8600 1450 50  0001 C CNN
-	1    8600 1450
+P 9450 1450
+F 0 "#PWR025" H 9450 1200 50  0001 C CNN
+F 1 "GND" H 9455 1277 50  0000 C CNN
+F 2 "" H 9450 1450 50  0001 C CNN
+F 3 "" H 9450 1450 50  0001 C CNN
+	1    9450 1450
 	1    0    0    -1
 $EndComp
@@
 Wire Wire Line
 	6800 4700 7550 4700
-NoConn ~ 7350 2350
 NoConn ~ 5200 2750
 NoConn ~ 8550 4600
@@
 F 0 "R1" V 2150 850 50  0000 C CNN
 F 1 "DNP" V 2250 850 50  0000 C CNN
-F 2 "Resistor_SMD:R_0603_1608Metric_Pad1.05x0.95mm_HandSolder" V 2180 850 50  0001 C CNN
+F 2 "humidity:R_0603_1608Metric_Pad1.05x0.95mm_HandSolder-DNP" V 2180 850 50  0001 C CNN
 F 3 "~" H 2250 850 50  0001 C CNN
 	1    2250 850
@@
 F 0 "R4" V 2150 1450 50  0000 C CNN
 F 1 "DNP" V 2250 1450 50  0000 C CNN
-F 2 "Resistor_SMD:R_0603_1608Metric_Pad1.05x0.95mm_HandSolder" V 2180 1450 50  0001 C CNN
+F 2 "humidity:R_0603_1608Metric_Pad1.05x0.95mm_HandSolder-DNP" V 2180 1450 50  0001 C CNN
 F 3 "~" H 2250 1450 50  0001 C CNN
 	1    2250 1450
@@
 NoConn ~ 5200 1750
 NoConn ~ 5200 1850
-NoConn ~ 5200 2350
 $Comp
 L power:GND #PWR07
@@
 L power:PWR_FLAG #FLG04
 U 1 1 5D226779
-P 8250 1750
-F 0 "#FLG04" H 8250 1825 50  0001 C CNN
-F 1 "PWR_FLAG" H 8250 1650 50  0000 C CNN
-F 2 "" H 8250 1750 50  0001 C CNN
-F 3 "~" H 8250 1750 50  0001 C CNN
-	1    8250 1750
-	1    0    0    -1
-$EndComp
-Wire Wire Line
-	7850 1800 8250 1800
-Wire Wire Line
-	8250 1800 8250 1750
-Connection ~ 7850 1800
-Wire Wire Line
-	7850 1800 7850 1850
+P 8150 650
+F 0 "#FLG04" H 8150 725 50  0001 C CNN
+F 1 "PWR_FLAG" H 8150 550 50  0000 C CNN
+F 2 "" H 8150 650 50  0001 C CNN
+F 3 "~" H 8150 650 50  0001 C CNN
+	1    8150 650
+	1    0    0    -1
+$EndComp
 Text Label 1400 1100 0    50   ~ 0
 FTDI_RX
@@
 F 0 "R12" V 6100 1800 50  0000 C CNN
 F 1 "DNP" V 6200 1800 50  0000 C CNN
-F 2 "Resistor_SMD:R_0603_1608Metric_Pad1.05x0.95mm_HandSolder" V 6130 1800 50  0001 C CNN
+F 2 "humidity:R_0603_1608Metric_Pad1.05x0.95mm_HandSolder-DNP" V 6130 1800 50  0001 C CNN
 F 3 "~" H 6200 1800 50  0001 C CNN
 	1    6200 1800
@@
 F 0 "R13" V 6350 1800 50  0000 C CNN
 F 1 "DNP" V 6450 1800 50  0000 C CNN
-F 2 "Resistor_SMD:R_0603_1608Metric_Pad1.05x0.95mm_HandSolder" V 6380 1800 50  0001 C CNN
+F 2 "humidity:R_0603_1608Metric_Pad1.05x0.95mm_HandSolder-DNP" V 6380 1800 50  0001 C CNN
 F 3 "~" H 6450 1800 50  0001 C CNN
 	1    6450 1800
@@
 LED1
 $Comp
-L humidity:D_Schottky_AncK D3
+L Device:D_Schottky D3
 U 1 1 5D01B3AF
-P 8250 900
-F 0 "D3" H 8250 1000 50  0000 R CNN
-F 1 "BAT54.215 " H 8250 800 50  0000 C CNN
-F 2 "Package_TO_SOT_SMD:SOT-23" H 8250 900 50  0001 C CNN
-F 3 "https://www.tme.eu/Document/2c1c71bcfe5aad5e582fdc49c2dc275f/BAT54.215.pdf" H 8250 900 50  0001 C CNN
-F 4 "https://www.tme.eu/se/en/details/bat54.215/smd-schottky-diodes/nexperia/" V 8250 900 50  0001 C CNN "TME Link"
-F 5 "0.22899" H 0   0   50  0001 C CNN "TME Price"
-	1    8250 900
-	1    0    0    -1
-$EndComp
-Wire Wire Line
-	8600 900  8400 900
-Wire Wire Line
-	7850 900  8100 900
-Wire Wire Line
-	7850 900  7850 1250
-Wire Wire Line
-	8600 1400 8600 1450
+P 9100 900
+F 0 "D3" H 9100 1000 50  0000 R CNN
+F 1 "B0520LW-7-F" H 9100 800 50  0000 C CNN
+F 2 "Diode_SMD:D_SOD-123" H 9100 900 50  0001 C CNN
+F 3 "https://www.tme.eu/Document/a7874355cfbb9c8a2b34695c20bc31e8/B0520LW.pdf" H 9100 900 50  0001 C CNN
+F 4 "https://www.tme.eu/se/en/details/b0520lw-7-f/smd-schottky-diodes/diodes-incorporated/" V 9100 900 50  0001 C CNN "TME Link"
+F 5 "0.50890" H 850 0   50  0001 C CNN "TME Price"
+	1    9100 900
+	1    0    0    -1
+$EndComp
+Wire Wire Line
+	9450 900  9250 900
+Wire Wire Line
+	8600 900  8950 900
+Wire Wire Line
+	9450 1400 9450 1450
 Wire Wire Line
 	2600 1050 2600 1100
@@
 Wire Wire Line
 	7100 3150 5200 3150
-Text Notes 5400 2850 0    50   ~ 0
-CS
-Text Notes 5400 2950 0    50   ~ 0
-MISO
-Text Notes 5400 3050 0    50   ~ 0
-MOSI
-Text Notes 5400 3150 0    50   ~ 0
-SCK
 Wire Wire Line
 	6700 4900 7550 4900
@@
 Text Label 6600 5700 0    50   ~ 0
 RFM_INT
-Text Label 8450 900  0    50   ~ 0
+Text Label 9300 900  0    50   ~ 0
 VBAT_IN
-Text Label 7850 1150 1    50   ~ 0
+Text Label 8650 900  0    50   ~ 0
 VBAT_D
 Text Label 7850 1750 1    50   ~ 0
@@
 Wire Wire Line
 	4500 1150 4500 1350
+$Comp
+L Device:C C7
+U 1 1 5D06EFEE
+P 8150 1400
+F 0 "C7" H 8200 1300 50  0000 L CNN
+F 1 "100n" V 8000 1400 50  0000 C CNN
+F 2 "Capacitor_SMD:C_0603_1608Metric_Pad1.05x0.95mm_HandSolder" H 8188 1250 50  0001 C CNN
+F 3 "~" H 8150 1400 50  0001 C CNN
+	1    8150 1400
+	1    0    0    -1
+$EndComp
+Wire Wire Line
+	8300 900  8150 900
+Wire Wire Line
+	8150 1250 8150 900
+Connection ~ 8150 900
+Wire Wire Line
+	8150 900  7850 900
+Wire Wire Line
+	8150 650  8150 900
+Wire Wire Line
+	7850 900  7850 1850
+$Comp
+L power:GND #PWR04
+U 1 1 5D08E603
+P 8150 1650
+F 0 "#PWR04" H 8150 1400 50  0001 C CNN
+F 1 "GND" H 8155 1477 50  0000 C CNN
+F 2 "" H 8150 1650 50  0001 C CNN
+F 3 "" H 8150 1650 50  0001 C CNN
+	1    8150 1650
+	1    0    0    -1
+$EndComp
+Wire Wire Line
+	8150 1550 8150 1650
+$Comp
+L Device:R R5
+U 1 1 5D093C3A
+P 6950 1800
+F 0 "R5" V 6850 1750 50  0000 L CNN
+F 1 "10k" V 6950 1800 50  0000 C CNN
+F 2 "Resistor_SMD:R_0603_1608Metric_Pad1.05x0.95mm_HandSolder" V 6880 1800 50  0001 C CNN
+F 3 "~" H 6950 1800 50  0001 C CNN
+	1    6950 1800
+	1    0    0    -1
+$EndComp
+Wire Wire Line
+	6950 1950 6950 2350
+Wire Wire Line
+	6950 2350 7350 2350
+$Comp
+L humidity:+3V3_PI #PWR02
+U 1 1 5D0991BC
+P 6950 1550
+F 0 "#PWR02" H 6950 1400 50  0001 C CNN
+F 1 "+3V3_PI" H 6965 1723 50  0000 C CNN
+F 2 "" H 6950 1550 50  0001 C CNN
+F 3 "" H 6950 1550 50  0001 C CNN
+	1    6950 1550
+	1    0    0    -1
+$EndComp
+Wire Wire Line
+	6950 1550 6950 1650
+Wire Wire Line
+	5200 2350 6950 2350
+Connection ~ 6950 2350
+Text Label 5800 2350 0    50   ~ 0
+MFP
+Text Label 6550 2850 0    50   ~ 0
+CS
+Text Label 6550 2950 0    50   ~ 0
+MISO
+Text Label 6550 3050 0    50   ~ 0
+MOSI
+Text Label 6550 3150 0    50   ~ 0
+SCK
 $EndSCHEMATC
