File: hardware/gateway/gateway.sch (KiCad schematic (older format))
At the start: 29 parts, among them J1 FTDI, J2 Conn_Coaxial, J3 Raspberry_Pi_2_3, U1 RFM69HW, U2 DS1307Z+, U3 AP130-xxY, Y1 32768

Commit message: Small udjustments to gateway PCB
Parts:
- gave numbers to parts that had none: 1
Changed lines of the file:
@@
 3V3_PI_17
 $Comp
-L Device:CP1 C?
+L Device:CP1 C4
 U 1 1 5D325ADD
 P 1150 4200
-F 0 "C?" H 1265 4246 50  0000 L CNN
+F 0 "C4" H 1265 4246 50  0000 L CNN
 F 1 "22u" H 1265 4155 50  0000 L CNN
 F 2 "Capacitor_SMD:CP_Elec_5x5.3" H 1150 4200 50  0001 C CNN
@@
 	1150 3900 1150 4050
 $Comp
-L power:GND #PWR?
+L power:GND #PWR04
 U 1 1 5D32BD4F
 P 1150 4400
-F 0 "#PWR?" H 1150 4150 50  0001 C CNN
+F 0 "#PWR04" H 1150 4150 50  0001 C CNN
 F 1 "GND" H 1155 4227 50  0000 C CNN
 F 2 "" H 1150 4400 50  0001 C CNN
